Commit message: Warehouse world (world:=warehouse), Gazebo + RViz by default, README update
- palletizer_gazebo/models/palletizer_warehouse: warehouse around the cell built in
  Blender from cell_config.yaml (OBJ visuals, 18 static collision boxes; roof/walls
  cast no shadows). Set dressing only: nothing inside the robot reach, pallet lane,
  conveyor, photo-eye beams or camera ROIs (tools/warehouse_blender/offline/wh_verify.py).
  Textured materials get Kd 1 (else Gazebo renders them black).
- world:=plain|warehouse on palletizer.launch.py and sim.launch.py; plain (default)
  is unchanged. GZ_SIM_RESOURCE_PATH via the env hook and the launch file.
- gui:=true is the launch default; scripted runs pass gui:=false.
- tools/warehouse_blender: build, export, render scripts and the keep-out verifier.
- README: Try it as copy-paste commands, warehouse world section (Gazebo frame),
  RViz screenshot, like-for-like throughput. RESULTS: both worlds' evaluations and RTF.

File: src/palletizer_gazebo/worlds/palletizing_cell.sdf.xacro (robot description, xacro)
@@ -2,5 +2,9 @@
 <!--
   Palletizing cell world. Rendered with xacro at launch time from cell_config.yaml:
-    xacro palletizing_cell.sdf.xacro cell_config:=<path> > palletizing_cell.sdf
+    xacro palletizing_cell.sdf.xacro cell_config:=<path> [environment:=plain|warehouse] > palletizing_cell.sdf
+  environment:=warehouse adds the palletizer_warehouse model (models/, built in Blender) around the
+  cell: set dressing only. It keeps out of the robot's reach, the pallet lane, the photo-eye
+  beams and the cameras' ROIs, and its roof/walls cast no shadows, so the lighting the cameras
+  see is unchanged. The ground collision is always this world's ground_plane.
   Conveyor pattern from gz-sim8 worlds/conveyor.sdf (TrackController on a static belt link).
   Collision shapes are plain boxes; visuals may be fancier.
@@ -9,4 +13,6 @@
   <xacro:arg name="cell_config" default=""/>
   <xacro:arg name="real_time_factor" default="1.0"/>
+  <xacro:arg name="environment" default="plain"/>
+  <xacro:property name="environment" value="$(arg environment)"/>
   <xacro:property name="cell" value="${xacro.load_yaml('$(arg cell_config)')}"/>
   <xacro:property name="cv" value="${cell['conveyor']}"/>
@@ -93,10 +99,20 @@
           <geometry><plane><normal>0 0 1</normal><size>20 20</size></plane></geometry>
         </collision>
-        <visual name="visual">
-          <geometry><plane><normal>0 0 1</normal><size>20 20</size></plane></geometry>
-          <xacro:material rgba="${[0.55, 0.55, 0.52, 1]}"/>
-        </visual>
-      </link>
-    </model>
+        <!-- warehouse: the floor visual comes with the warehouse model (same mean colour) -->
+        <xacro:if value="${environment == 'plain'}">
+          <visual name="visual">
+            <geometry><plane><normal>0 0 1</normal><size>20 20</size></plane></geometry>
+            <xacro:material rgba="${[0.55, 0.55, 0.52, 1]}"/>
+          </visual>
+        </xacro:if>
+      </link>
+    </model>
+    <xacro:if value="${environment == 'warehouse'}">
+      <include>
+        <uri>model://palletizer_warehouse</uri>
+        <name>warehouse</name>
+        <pose>0 0 0 0 0 0</pose>
+      </include>
+    </xacro:if>
     <!-- ============================ Conveyor ============================ -->
     <xacro:property name="cv_len" value="${cv['x_end'] - cv['x_start']}"/>

Commit message: PalletMover: carried stack stays level; photo-eye posts; GIF re-recorded
- PalletMover also commands every carried link's velocity each step (the conveyor
  velocity, no rotation; zero on the last step). With pose commands alone, gravity
  accumulated between teleports and the boxes of a moving stack sank / tilted in the
  render (side camera: stepped top at 1.0-1.5 m into the exit; now flat), while
  /sim/box_poses (model poses = the commanded pose) showed 0.0 mm.
- World: the photo-eye emitters / reflectors stand on posts with floor plates (visual
  only, inside each head's footprint, below the beam and min_object_height).
- warehouse_demo.gif re-recorded with both fixes (24-box pallet, 8 per layer).

Checked: run_all.sh (all 7 pass; pallet mover: rigid ride 0.4 mm, overhang still
tips, shoved box stays, box rests on the new deck), eval_perception 68/68,
eval_pallet_perception 9/9, pick_place_test 20/20.

File: src/palletizer_gazebo/worlds/palletizing_cell.sdf.xacro (robot description, xacro)
@@ -214,4 +214,23 @@
               <xacro:material rgba="${[0.9, 0.1, 0.1, 1]}"/>
             </visual>
+            <!-- Posts and floor plates under both heads (visual only, like the heads). Each post
+                 stays inside its head's footprint (the overhead camera sees only the head), ends
+                 under the head (below the beam and below min_object_height above the belt). -->
+            <xacro:property name="eye_z" value="${cv['belt_top_z'] + eye['height']}"/>
+            <xacro:property name="post_h" value="${eye_z - 0.025}"/>
+            <xacro:macro name="eye_post" params="name x sx sy">
+              <visual name="${name}_post">
+                <pose>${x} 0 ${-0.025 - post_h / 2} 0 0 0</pose>
+                <geometry><box><size>${sx} ${sy} ${post_h}</size></box></geometry>
+                <xacro:material rgba="${[0.2, 0.22, 0.25, 1]}"/>
+              </visual>
+              <visual name="${name}_foot">
+                <pose>${x} 0 ${0.005 - eye_z} 0 0 0</pose>
+                <geometry><box><size>0.10 0.10 0.01</size></box></geometry>
+                <xacro:material rgba="${[0.2, 0.22, 0.25, 1]}"/>
+              </visual>
+            </xacro:macro>
+            <xacro:eye_post name="emitter" x="0" sx="0.02" sy="0.02"/>
+            <xacro:eye_post name="reflector" x="${cv['belt_width'] + 2 * eye['offset']}" sx="0.008" sy="0.03"/>
             <sensor name="eye_${z['name']}" type="gpu_lidar">
               <always_on>true</always_on>
